File: FINISHED/SOUND_SOURCE/SOUND_SOURCE_modular_PCB/SOUND_SOURCE_modular/SOUND_SOURCE_modular.sch (KiCad schematic (older format))
At the start: 82 parts, among them J1 AUDIO_OUT, J10 GATE_INPUT, J2 POWER, J3 Front Panel conn, J4 Front panel conn, J5 CV_INPUT, J6 FM_INPUT, J7 TIMBRE CV, J8 COLOR CV, Q1 BC547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

Commit message: sound source circuit fix cv anf fm inputs. increase capacitor
Parts:
- C12, C13: value 220pF -> 10nF
Changed lines of the file:
@@
 P 1700 6400
 F 0 "C12" H 1750 6500 50  0000 L CNN
-F 1 "220pF" H 1750 6300 50  0000 L CNN
+F 1 "10nF" H 1750 6300 50  0000 L CNN
 F 2 "Capacitors_ThroughHole:C_Disc_D4.3mm_W1.9mm_P5.00mm" H 1738 6250 50  0001 C CNN
 F 3 "~" H 1700 6400 50  0001 C CNN
@@
 P 3700 6400
 F 0 "C13" H 3750 6500 50  0000 L CNN
-F 1 "220pF" H 3750 6300 50  0000 L CNN
+F 1 "10nF" H 3750 6300 50  0000 L CNN
 F 2 "Capacitors_ThroughHole:C_Disc_D4.3mm_W1.9mm_P5.00mm" H 3738 6250 50  0001 C CNN
 F 3 "~" H 3700 6400 50  0001 C CNN
