File: FINISHED/SEQUENCER/SEQUENCER_modular_PCB/SEQUENCER_modular/SEQUENCER_modular.sch (KiCad schematic (older format))
At the start: 60 parts, among them IC1 LM336, J1 POWER, J10 AFTER_TOUCH_OUT, J11 POTS_POWER, J12 CV_OUT, J2 EXT_RST_IN, J3 LEDS, J4 EXT_CLK_IN, J5 MIDI_IN, J6 ENCODER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

Commit message: VCF project
Parts:
- IC1: symbol LM336:LM336 -> SEQUENCER_modular-rescue:LM336-LM336
Other:
- note added: "2: MIDI_PIN5\n1: MIDI_PIN4"
- note removed: "2: MIDI_PIN4\n1: MIDI_PIN5"
Changed lines of the file:
@@
 Connection ~ 4350 1700
 Text Notes 3550 1200 0    50   ~ 0
-2: MIDI_PIN4\n1: MIDI_PIN5
+2: MIDI_PIN5\n1: MIDI_PIN4
 Text GLabel 5550 1450 2    50   Input ~ 0
 MIDI_IN_RX
@@
 	8450 1750 8450 1700
 $Comp
-L LM336:LM336 IC1
+L SEQUENCER_modular-rescue:LM336-LM336 IC1
 U 1 1 5EDB848E
 P 6400 1650
